File: emboard.sch (KiCad schematic (older format))
At the start: 2 parts, among them P1 2pin-header, P2 2pin-header

Commit message: add buttons
Parts:
- added P3, P4: 2pin-header, footprints:2pin-header, symbol 2pin-header
Connections:
- new net Buttonleft1: P3.2
- new net Buttonleft2: P3.1
- new net buttonright1: P4.2
- new net buttonright2: P4.1
Changed lines of the file:
@@
 LIBS:valves
 LIBS:2pin-header
+LIBS:emboard-cache
 EELAYER 25 0
 EELAYER END
@@
 Wire Wire Line
 	4200 4500 4150 4500
+$Comp
+L 2pin-header P3
+U 1 1 57D894F6
+P 4350 1400
+F 0 "P3" H 4350 1500 60  0000 C CNN
+F 1 "2pin-header" H 4350 1400 60  0000 C CNN
+F 2 "footprints:2pin-header" H 4350 1400 60  0001 C CNN
+F 3 "" H 4350 1400 60  0001 C CNN
+	1    4350 1400
+	1    0    0    -1
+$EndComp
+Text GLabel 4150 2100 0    60   Input ~ 0
+Buttonleft1
+Text GLabel 6650 2150 0    60   Input ~ 0
+buttonright1
+$Comp
+L 2pin-header P4
+U 1 1 57D89823
+P 6650 1400
+F 0 "P4" H 6650 1500 60  0000 C CNN
+F 1 "2pin-header" H 6650 1400 60  0000 C CNN
+F 2 "footprints:2pin-header" H 6650 1400 60  0001 C CNN
+F 3 "" H 6650 1400 60  0001 C CNN
+	1    6650 1400
+	1    0    0    -1
+$EndComp
+Text GLabel 4550 2300 0    60   Input ~ 0
+Buttonleft2
+Text GLabel 7050 2400 0    60   Input ~ 0
+buttonright2
+Wire Wire Line
+	4150 2100 4150 1900
+Wire Wire Line
+	4150 1900 4100 1900
+Wire Wire Line
+	4550 2300 4550 1900
+Wire Wire Line
+	4550 1900 4450 1900
+Wire Wire Line
+	6650 2150 6650 1900
+Wire Wire Line
+	6650 1900 6400 1900
+Wire Wire Line
+	6750 1900 7050 1900
+Wire Wire Line
+	7050 1900 7050 2400
 $EndSCHEMATC
